File: v0_miniAB_pancake_board.kicad_pcb (KiCad board)
At the start: 2 copper layers, 51 x 37.4 mm, 13 parts, among them J1 Conn_01x04_Female, J10 Conn_01x03_Female, J11 Conn_01x03_Female, J2 Conn_01x02_Female, J3 Conn_01x02_Female, J4 Conn_01x02_Female, J5 Conn_01x02_Female, J6 Conn_01x02_Female, J7 Conn_01x03_Female, J8 Conn_01x03_Female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

Commit message: a little bit more clearance around the mounting holes
Routing:
- net /VFAN0: track 82.0 -> 83.1 mm
